File: 02_LED-Einheit/Prints/led_print_eckig/led_print_V2.kicad_pcb (KiCad board)
At the start: 2 copper layers, 125 x 25.7 mm, 18 parts, among them J1 Conn_01x02_Pin

Commit message: small_changes_readmes
Parts:
- J1: footprint Connector_PinHeader_2.54mm:PinHeader_1x02_P2.54mm_Vertical -> Connector_PinHeader_2.54mm:PinHeader_1x02_P2.54mm_Horizontal
- moved J1 14.5 mm to (77.0, 64.8), turned to 180 degrees
- moved R1 12.7 mm to (68.1, 70.1), turned to 0 degrees
Connections:
- J1 pad 1: Net-(D1-A) -> Net-(J1-Pin_1)
- R1 pad 1: Net-(D1-A) -> Net-(J1-Pin_1)
- R1 pad 2: GND -> Net-(D1-A)
Routing:
- net Net-(J1-Pin_1): track 0.00 -> 12.9 mm
- net Net-(D1-A): track 221.3 -> 211.5 mm
