File: 01_Touch-Sensorik/Prints/Schreibtischlampe_V5.kicad_pcb (KiCad board)
At the start: 2 copper layers, 64.8 x 57.1 mm, 26 parts, among them J1 Versorgung, J2 Lampenkopf, J5 Messpunkte, Q1 BC547, Q2 BC547, Q3 BDX53BG, U1 NE555P, U2 4017

Commit message: changes documentation
Parts:
- C1: footprint Capacitor_THT:CP_Radial_D4.0mm_P1.50mm -> Capacitor_THT:CP_Radial_D4.0mm_P2.00mm
- J1: footprint TerminalBlock_Phoenix:TerminalBlock_Phoenix_MKDS-1,5-2-5.08_1x02_P5.08mm_Horizontal -> TerminalBlock_Phoenix:TerminalBlock_Phoenix_MKDS-1,5-2_1x02_P5.00mm_Horizontal
- J2: footprint TerminalBlock_Phoenix:TerminalBlock_Phoenix_MKDS-1,5-3-5.08_1x03_P5.08mm_Horizontal -> TerminalBlock_Phoenix:TerminalBlock_Phoenix_MKDS-1,5-3_1x03_P5.00mm_Horizontal
Routing:
- net GND: track 1.91 -> 0.00 mm
Other:
- board text added: "${REVISION}"
- board text added: "${TITLE}"
- board text added: "HTL Steyr"
