File: 01_Touch-Sensorik/Prints/Schreibtischlampe_V5.kicad_sch (KiCad schematic)
At the start: 26 parts, among them J1 Versorgung, J2 Lampenkopf, J5 Messpunkte, Q1 BC547, Q2 BC547, Q3 BDX53BG, U1 NE555P, U2 4017

Commit message: changes documentation
Parts:
- C1: footprint Capacitor_THT:CP_Radial_D4.0mm_P1.50mm -> Capacitor_THT:CP_Radial_D4.0mm_P2.00mm; Preis/Stück [€] (none) -> 0,09; RS/URL https://at.rs-online.com/web/p/aluminium-elektrolytkondensa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 -> (none); Stück (none) -> 100; URL (none) -> https://at.rs-online.com/web/p/aluminium-elektrolytkondensa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
- C2, C3: Preis/Stück [€] (none) -> 0,166; RS/URL https://at.rs-online.com/web/p/keramik-vielschichtkondensat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 -> (none); Stück (none) -> 250; URL (none) -> https://at.rs-online.com/web/p/keramik-vielschichtkondensat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
- D1, D2, D3: Preis/Stück [€] (none) -> 0,026; RS/URL https://at.rs-online.com/web/p/schottky-dioden-und-gleichri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 -> (none); Stück (none) -> 500; URL (none) -> https://at.rs-online.com/web/p/schottky-dioden-und-gleichri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
- H1, H2, H3, H4: Bestellnummer (none) -> -; Lieferant  (none) -> -; Preis/Stück [€] (none) -> -; Stück (none) -> -; URL (none) -> -
- J1: footprint TerminalBlock_Phoenix:TerminalBlock_Phoenix_MKDS-1,5-2-5.08_1x02_P5.08mm_Horizontal -> TerminalBlock_Phoenix:TerminalBlock_Phoenix_MKDS-1,5-2_1x02_P5.00mm_Horizontal; Bestellnummer (none) -> 731091 - 62; Lieferant  (none) -> Conrad; Preis/Stück [€] (none) -> 0,284; Stück (none) -> 30; URL (none) -> https://www.conrad.at/de/p/degson-dg301-5-0-02p-12-schraubk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
- J2: footprint TerminalBlock_Phoenix:TerminalBlock_Phoenix_MKDS-1,5-3-5.08_1x03_P5.08mm_Horizontal -> TerminalBlock_Phoenix:TerminalBlock_Phoenix_MKDS-1,5-3_1x03_P5.00mm_Horizontal; Bestellnummer (none) -> 730196 - 62; Lieferant  (none) -> Conrad; Preis/Stück [€] (none) -> 0,41; Stück (none) -> 30; URL (none) -> https://www.conrad.at/de/p/degson-dg301-5-0-03p-12-schraubk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
- J5, R1, R2, R3, R5, U_Netzteil1: Bestellnummer (none) -> -; Lieferant  (none) -> HTL; Preis/Stück [€] (none) -> -; Stück (none) -> -; URL (none) -> -
- Q1, Q2: Preis/Stück [€] (none) -> 0,099; RS/URL https://at.rs-online.com/web/p/bipolare-transistoren/7619822 -> (none); Stück (none) -> 100; URL (none) -> https://at.rs-online.com/web/p/bipolare-transistoren/7619822
- Q3: Preis/Stück [€] (none) -> 0,774; RS/URL https://at.rs-online.com/web/p/bipolare-transistoren/186793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 -> (none); Stück (none) -> 3 * 10; URL (none) -> https://at.rs-online.com/web/p/bipolare-transistoren/186793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
- RV1, RV4: Preis/Stück [€] (none) -> 0,33; RS/URL https://www.conrad.at/de/p/piher-pt10lv10-103a2020-pm-s-pt1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 -> (none); Stück (none) -> 30; URL (none) -> https://www.conrad.at/de/p/piher-pt10lv10-103a2020-pm-s-pt1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
- RV2: Preis/Stück [€] (none) -> 0,33; RS/URL https://www.conrad.at/de/p/piher-pt10lv10-505a2020-pm-s-pt1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 -> (none); Stück (none) -> 30; URL (none) -> https://www.conrad.at/de/p/piher-pt10lv10-505a2020-pm-s-pt1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
- U1: Preis/Stück [€] (none) -> 1,15; RS/URL https://at.rs-online.com/web/p/operationsverstarker/4363046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 -> (none); Stück (none) -> 30; URL (none) -> https://at.rs-online.com/web/p/operationsverstarker/4363046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
- U2: Preis/Stück [€] (none) -> 0,92; RS/URL https://at.farnell.com/texas-instruments/cd4017be/z-hler-de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 -> (none); Stück (none) -> 30; URL (none) -> https://at.farnell.com/texas-instruments/cd4017be/z-hler-de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
